Commit message: It heckin works correctly now

File: catkin_ws/src/me212arm/model/me212arm.xacro (robot description, xacro)
@@ -51,7 +51,7 @@
     <parent link="arm_base"/>
     <child link="link1"/>
-    <origin xyz="0 0 0"/>
+    <origin xyz="0 0 0" rpy="0 ${-M_PI/2} ${M_PI}"/>
     <limit effort="300" lower="${-M_PI}" upper="${M_PI/2}" velocity="7.33"/>
-    <axis xyz="0 1 0"/>
+    <axis xyz="0 -1 0"/>
 </joint>
 <joint name="joint2" type="revolute">
@@ -60,5 +60,5 @@
     <origin xyz="0 0 ${link1_length}" />
     <limit effort="300" lower="${-M_PI}" upper="${M_PI}" velocity="7.33"/>
-    <axis xyz="0 1 0"/>
+    <axis xyz="0 -1 0"/>
 </joint>
 <joint name="joint3" type="fixed">

File: catkin_ws/src/me212bot/model/me212bot.xacro (robot description, xacro)
@@ -7,5 +7,5 @@
         <parent link="robot_base"/>
         <child link="arm_base"/>
-    <origin xyz="0.1 0.222 0.25"  rpy="0 ${M_PI/2} 0"/>
+    <origin xyz="0.05 0.222 0.25"  rpy="0 0 0"/>
     </joint>
 </robot>
